File: flight-pcb/flight-pcb.sch (KiCad schematic (older format))
At the start: 21 parts, among them J1 Conn_01x05, J2 Conn_01x06, J3 Conn_01x08, J4 Conn_01x20, J5 Conn_01x20, J6 Conn_01x05, J7 Conn_01x07, J8 Conn_01x02

Commit message: updated project to KiCad V6.0
Parts:
- D1: PNUM (none) -> QBLP601-AG15
- D2: PNUM (none) -> QBLP601-R5
- D3: PNUM (none) -> QBLP601-Y5
- D4: PNUM (none) -> LTST-C193TBKT-5A
- D5: PNUM (none) -> PMEG2005EH,115
- R1: PNUM (none) -> RMCF0603FT270R
- R2: PNUM (none) -> 850-RMCF0603FT309RCT-ND
- R3: PNUM (none) -> RMCF0603FT294R
- R4: PNUM (none) -> RMCF0603FT100R
Other:
- note added: "SPI SMT SD Card"
- moved on the sheet: D1, D2, D3, D4, H1, H2, H3, H4, R1, R2, R3, R4
