File: flight-pcb/flight-pcb.kicad_pcb (KiCad board)
At the start: 2 copper layers, 88.8 x 51.3 mm, 21 parts, among them J1 Conn_01x05, J2 Conn_01x06, J3 Conn_01x08, J4 Conn_01x20, J5 Conn_01x20, J6 Conn_01x05, J7 Conn_01x07, J8 Conn_01x02

Commit message: updated project to KiCad V6.0
Other:
- net class Default removed

Commit message: updated raspberry pi header pins
updated board to include new library with different pin numbers
Parts:
- removed J5: Conn_01x20, Connector_PinHeader_2.54mm:PinHeader_1x20_P2.54mm_Vertical
- added J9: Conn_01x20_v2, Library:PinHeader_1x20_v2_P2.54mm_Vertical, F.Cu at (143.5, 73.7)
- R1: value 68 -> 270
- R2: value 68 -> 309
- R3: value 68 -> 294
- R4: value 68 -> 100
Connections:
- net Net-(J4-Pad12) renamed GP9
- net Net-(J4-Pad14) renamed GP10
- net Net-(J4-Pad15) renamed GP11
- net Net-(J4-Pad16) renamed GP12
- net Net-(J4-Pad17) renamed GP13
- net Net-(J4-Pad19) renamed GP14
- net Net-(J4-Pad20) renamed GP15
- J1 pad 2: Net-(J1-Pad2) -> unconnected-(J1-Pad2)
- J2 pad 2: Net-(J2-Pad2) -> unconnected-(J2-Pad2)
- J2 pad 6: Net-(J2-Pad6) -> unconnected-(J2-Pad6)
- J3 pad 2: Net-(J3-Pad2) -> unconnected-(J3-Pad2)
- J3 pad 5: Net-(J3-Pad5) -> unconnected-(J3-Pad5)
- J3 pad 7: Net-(J3-Pad7) -> unconnected-(J3-Pad7)
- J3 pad 8: Net-(J3-Pad8) -> unconnected-(J3-Pad8)
- J4 pad 7: Net-(J4-Pad7) -> unconnected-(J4-Pad7)
- J6 pad 1: Net-(J6-Pad1) -> unconnected-(J6-Pad1)
- J6 pad 3: Net-(J6-Pad3) -> unconnected-(J6-Pad3)
- J6 pad 4: Net-(J6-Pad4) -> unconnected-(J6-Pad4)
- J6 pad 5: Net-(J6-Pad5) -> unconnected-(J6-Pad5)
- J7 pad 2: Net-(J7-Pad2) -> unconnected-(J7-Pad2)
- J8 pad 1: Net-(D5-Pad2) -> GND
- J8 pad 2: GND -> Net-(D5-Pad2)
